Commit message: test run simple_thruster with visual

File: src/ex_mm40b3_description/urdf/ex_mm40b3.xacro (robot description, xacro)
@@ -4,4 +4,5 @@
 <xacro:include filename="$(find ex_mm40b3_description)/urdf/ex_mm40b3.trans" />
 <xacro:include filename="$(find ex_mm40b3_description)/urdf/ex_mm40b3.gazebo" />
+<!-- <xacro:include filename="$(find ex_mm40b3_description)/urdf/plugins.gazebo"/> -->
 <link name="base_link">
   <inertial>

File: src/launcher20deg_description/launcher20deg.urdf (robot description, URDF)
Before this commit: robot launcher20deg, 6 links, 5 joints
Links:
- added link Cup_3, mass 132.23344015308516; collision mesh filename=package://launcher20deg_description/meshes/Cup_3.stl scale=0.001 0.001 0.001; visual mesh filename=package://launcher20deg_description/meshes/Cup_3.stl scale=0.001 0.001 0.001
Joints:
- added joint CupOpener: type revolute, parent Canister_1, child Cup_3, origin xyz=1.546373 0.0 0.232105 rpy=0 0 0, axis 0.0 1.0 0.0, limit lower=0.0 upper=4.712389 effort=100 velocity=100

File: src/launcher20deg_description/urdf/launcher20deg.xacro (robot description, xacro)
@@ -50,5 +50,5 @@
   </collision>
 </link>
-<!-- <link name="Cup_3">
+<link name="Cup_3">
   <inertial>
     <origin xyz="-0.1113901774930488 -2.4584670189393287e-09 0.29080423143479095" rpy="0 0 0"/>
@@ -69,5 +69,5 @@
     </geometry>
   </collision>
-</link> -->
+</link>
 <link name="Cup_1">
   <inertial>
@@ -135,5 +135,5 @@
   <child link="Canister_1"/>
 </joint>
-<!-- <joint name="CupOpener" type="revolute">
+<joint name="CupOpener" type="revolute">
   <origin xyz="1.546373 0.0 0.232105" rpy="0 0 0"/>
   <parent link="Canister_1"/>
@@ -141,5 +141,5 @@
   <axis xyz="0.0 1.0 0.0"/>
   <limit upper="4.712389" lower="0.0" effort="100" velocity="100"/>
-</joint> -->
+</joint>
 <joint name="CupCloser" type="fixed">
   <origin xyz="-4.439955 0.0 -0.859884" rpy="0 0 0"/>
