Commit message: edit vector visualization

File: src/ssm_models/mm40b3_description/urdf/materials.xacro (robot description, xacro)
@@ -1,6 +1,30 @@
 <?xml version="1.0" ?>
 <robot name="mm40b3" xmlns:xacro="http://www.ros.org/wiki/xacro" >
-<material name="silver">
-  <color rgba="0.700 0.700 0.700 1.000"/>
-</material>
+  <material name="grey">
+    <color rgba="${211/256} ${211/256} ${211/256} 1.0"/>
+  </material>
+  <material name="darkgrey">
+    <color rgba="${47/255} ${79/255} ${79/255} 1.000"/>
+  </material>
+  <material name="silver">
+    <color rgba="0.700 0.700 0.700 1.000"/>
+  </material>
+  <material name="white">
+    <color rgba="1 1 1 1" />
+  </material>
+  <material name="orange">
+    <color rgba="1 0.3 0.1 1"/>
+  </material>
+  <material name="blue">
+    <color rgba="0.2 0.2 1 1"/>
+  </material>
+  <material name="red">
+    <color rgba="0.8 0 0 1"/>
+  </material>
+  <material name="green">
+    <color rgba="0.0 1 0.0 1"/>
+  </material>
+  <material name="black">
+    <color rgba="0 0 0 1"/>
+  </material>
 </robot>

File: src/ssm_models/mm40b3_description/urdf/mm40b3.xacro (robot description, xacro)
@@ -15,5 +15,5 @@
       <mesh filename="package://mm40b3_description/meshes/base_link.stl" scale="0.001 0.001 0.001"/>
     </geometry>
-    <material name="silver"/>
+    <material name="white"/>
   </visual>
   <collision>
@@ -35,5 +35,5 @@
       <mesh filename="package://mm40b3_description/meshes/FinHolder_1.stl" scale="0.001 0.001 0.001"/>
     </geometry>
-    <material name="silver"/>
+    <material name="blue"/>
   </visual>
   <collision>
@@ -55,5 +55,5 @@
       <mesh filename="package://mm40b3_description/meshes/FinHolder_4.stl" scale="0.001 0.001 0.001"/>
     </geometry>
-    <material name="silver"/>
+    <material name="blue"/>
   </visual>
   <collision>
@@ -75,5 +75,5 @@
       <mesh filename="package://mm40b3_description/meshes/FinHolder_3.stl" scale="0.001 0.001 0.001"/>
     </geometry>
-    <material name="silver"/>
+    <material name="blue"/>
   </visual>
   <collision>
@@ -95,5 +95,5 @@
       <mesh filename="package://mm40b3_description/meshes/FinHolder_2.stl" scale="0.001 0.001 0.001"/>
     </geometry>
-    <material name="silver"/>
+    <material name="blue"/>
   </visual>
   <collision>
@@ -115,5 +115,5 @@
       <mesh filename="package://mm40b3_description/meshes/Wing1_1.stl" scale="0.001 0.001 0.001"/>
     </geometry>
-    <material name="silver"/>
+    <material name="orange"/>
   </visual>
   <collision>
@@ -135,5 +135,5 @@
       <mesh filename="package://mm40b3_description/meshes/Booster_1.stl" scale="0.001 0.001 0.001"/>
     </geometry>
-    <material name="silver"/>
+    <material name="grey"/>
   </visual>
   <collision>
@@ -155,5 +155,5 @@
       <mesh filename="package://mm40b3_description/meshes/Wing1_2.stl" scale="0.001 0.001 0.001"/>
     </geometry>
-    <material name="silver"/>
+    <material name="orange"/>
   </visual>
   <collision>
@@ -175,5 +175,5 @@
       <mesh filename="package://mm40b3_description/meshes/Wing1_3.stl" scale="0.001 0.001 0.001"/>
     </geometry>
-    <material name="silver"/>
+    <material name="orange"/>
   </visual>
   <collision>
@@ -195,5 +195,5 @@
       <mesh filename="package://mm40b3_description/meshes/Wing1_4.stl" scale="0.001 0.001 0.001"/>
     </geometry>
-    <material name="silver"/>
+    <material name="orange"/>
   </visual>
   <collision>
@@ -215,5 +215,5 @@
       <mesh filename="package://mm40b3_description/meshes/Holder_1.stl" scale="0.001 0.001 0.001"/>
     </geometry>
-    <material name="silver"/>
+    <material name="darkgrey"/>
   </visual>
   <collision>
@@ -235,5 +235,5 @@
       <mesh filename="package://mm40b3_description/meshes/Holder_2.stl" scale="0.001 0.001 0.001"/>
     </geometry>
-    <material name="silver"/>
+    <material name="darkgrey"/>
   </visual>
   <collision>
@@ -255,5 +255,5 @@
       <mesh filename="package://mm40b3_description/meshes/Holder_3.stl" scale="0.001 0.001 0.001"/>
     </geometry>
-    <material name="silver"/>
+    <material name="darkgrey"/>
   </visual>
   <collision>
@@ -275,5 +275,5 @@
       <mesh filename="package://mm40b3_description/meshes/Holder_4.stl" scale="0.001 0.001 0.001"/>
     </geometry>
-    <material name="silver"/>
+    <material name="darkgrey"/>
   </visual>
   <collision>
@@ -295,5 +295,5 @@
       <mesh filename="package://mm40b3_description/meshes/Fin_1.stl" scale="0.001 0.001 0.001"/>
     </geometry>
-    <material name="silver"/>
+    <material name="orange"/>
   </visual>
   <collision>
@@ -315,5 +315,5 @@
       <mesh filename="package://mm40b3_description/meshes/Fin_2.stl" scale="0.001 0.001 0.001"/>
     </geometry>
-    <material name="silver"/>
+    <material name="orange"/>
   </visual>
   <collision>
@@ -335,5 +335,5 @@
       <mesh filename="package://mm40b3_description/meshes/Fin_3.stl" scale="0.001 0.001 0.001"/>
     </geometry>
-    <material name="silver"/>
+    <material name="orange"/>
   </visual>
   <collision>
@@ -355,5 +355,5 @@
       <mesh filename="package://mm40b3_description/meshes/Fin_4.stl" scale="0.001 0.001 0.001"/>
     </geometry>
-    <material name="silver"/>
+    <material name="orange"/>
   </visual>
   <collision>
@@ -459,9 +459,10 @@
   <limit upper="2.146755" lower="0.0" effort="100" velocity="100"/>
 </joint>
-<joint name="fin_fold3" type="continuous">
+<joint name="fin_fold3" type="revolute">
   <origin xyz="0.0 -0.038891 -0.038891" rpy="0 0 0"/>
   <parent link="FinHolder_3"/>
   <child link="Fin_3"/>
   <axis xyz="1.0 -0.0 -0.0"/>
+  <limit upper="2.146755" lower="0.0" effort="100" velocity="100"/>
 </joint>
 <joint name="fin_fold4" type="revolute">
