Commit message: deflection effect in aerodynamic plugin

File: src/ssm_models/model_missile_description/model_missile.urdf (robot description, URDF)
Before this commit: robot model_missile, 13 links, 12 joints
Links:
- added link Booster_1, mass 120.00001114591107; collision mesh filename=package://model_missile_description/meshes/Booster_1.stl scale=0.001 0.001 0.001; visual mesh filename=package://model_missile_description/meshes/Booster_1.stl scale=0.001 0.001 0.001
- added link Holder_1, mass 13.50000107858645; collision mesh filename=package://model_missile_description/meshes/Holder_1.stl scale=0.001 0.001 0.001; visual mesh filename=package://model_missile_description/meshes/Holder_1.stl scale=0.001 0.001 0.001
- added link Holder_2, mass 13.50000107858645; collision mesh filename=package://model_missile_description/meshes/Holder_2.stl scale=0.001 0.001 0.001; visual mesh filename=package://model_missile_description/meshes/Holder_2.stl scale=0.001 0.001 0.001
- added link Holder_3, mass 13.50000107858645; collision mesh filename=package://model_missile_description/meshes/Holder_3.stl scale=0.001 0.001 0.001; visual mesh filename=package://model_missile_description/meshes/Holder_3.stl scale=0.001 0.001 0.001
- added link Holder_4, mass 13.50000107858645; collision mesh filename=package://model_missile_description/meshes/Holder_4.stl scale=0.001 0.001 0.001; visual mesh filename=package://model_missile_description/meshes/Holder_4.stl scale=0.001 0.001 0.001
Joints:
- added joint HolderJoint1: type fixed, parent base_link, child Holder_1, origin xyz=1.375615 0.132493 0.132493 rpy=0 0 0
- added joint HolderJoint2: type fixed, parent base_link, child Holder_2, origin xyz=1.375615 -0.132493 0.132493 rpy=0 0 0
- added joint HolderJoint3: type fixed, parent base_link, child Holder_3, origin xyz=1.375615 -0.132493 -0.132493 rpy=0 0 0
- added joint HolderJoint4: type fixed, parent base_link, child Holder_4, origin xyz=1.375615 0.132493 -0.132493 rpy=0 0 0
- added joint booster_fixing: type fixed, parent base_link, child Booster_1, origin xyz=-1.880856 0.0 0.0 rpy=0 0 0

File: src/ssm_models/model_missile_description/urdf/model_missile.xacro (robot description, xacro)
@@ -1,6 +1,6 @@
 <?xml version="1.0" ?>
 <robot name="model_missile" xmlns:xacro="http://www.ros.org/wiki/xacro">
-<xacro:property name="use_booster" value="true"/>
-<xacro:property name="use_holder" value="true"/>
+<xacro:property name="use_booster" value="false"/>
+<xacro:property name="use_holder" value="false"/>
 <xacro:include filename="$(find model_missile_description)/urdf/materials.xacro" />
 <xacro:include filename="$(find model_missile_description)/urdf/model_missile.trans" />

Commit message: able to set initial position

File: src/ssm_models/model_missile_description/model_missile.urdf (robot description, URDF)
Before this commit: robot model_missile, 18 links, 17 joints
Links:
- removed link Booster_1
- removed link Holder_1
- removed link Holder_2
- removed link Holder_3
- removed link Holder_4
Joints:
- removed joint HolderJoint1
- removed joint HolderJoint2
- removed joint HolderJoint3
- removed joint HolderJoint4
- removed joint booster_fixing
- joint fins_rev1: limit lower=-0.349066 upper=0.349066 effort=100 velocity=100 -> lower=-0.349066 upper=0.349066 effort=1000 velocity=100
- joint fins_rev2: limit lower=-0.349066 upper=0.349066 effort=100 velocity=100 -> lower=-0.349066 upper=0.349066 effort=1000 velocity=100
- joint fins_rev3: limit lower=-0.349066 upper=0.349066 effort=100 velocity=100 -> lower=-0.349066 upper=0.349066 effort=1000 velocity=100
- joint fins_rev4: limit lower=-0.349066 upper=0.349066 effort=100 velocity=100 -> lower=-0.349066 upper=0.349066 effort=1000 velocity=100

File: src/ssm_models/model_missile_description/urdf/model_missile.xacro (robot description, xacro)
@@ -3,4 +3,6 @@
 <xacro:property name="use_booster" value="false"/>
 <xacro:property name="use_holder" value="false"/>
+<xacro:property name="foldable" value="true"/>
+<xacro:property name="deflection" value="true"/>
 <xacro:include filename="$(find model_missile_description)/urdf/materials.xacro" />
 <xacro:include filename="$(find model_missile_description)/urdf/model_missile.trans" />
@@ -377,100 +379,156 @@
   </joint>
 </xacro:if>
-<joint name="fins_rev1" type="revolute">
-<!-- <joint name="fins_rev1" type="fixed"> -->
-  <origin xyz="-1.700844 0.127279 0.127279" rpy="0 0 0"/>
-  <parent link="base_link"/>
-  <child link="FinHolder_1"/>
-  <axis xyz="-0.0 0.707107 0.707107"/>
-  <limit upper="0.349066" lower="-0.349066" effort="1000" velocity="100"/>
-</joint>
-<joint name="fins_rev2" type="revolute">
-<!-- <joint name="fins_rev2" type="fixed"> -->
-  <origin xyz="-1.700844 0.127279 -0.127279" rpy="0 0 0"/>
-  <parent link="base_link"/>
-  <child link="FinHolder_2"/>
-  <axis xyz="-0.0 0.707107 -0.707107"/>
-  <limit upper="0.349066" lower="-0.349066" effort="1000" velocity="100"/>
-</joint>
-<joint name="fins_rev3" type="revolute">
-<!-- <joint name="fins_rev3" type="fixed"> -->
-  <origin xyz="-1.700844 -0.127279 -0.127279" rpy="0 0 0"/>
-  <parent link="base_link"/>
-  <child link="FinHolder_3"/>
-  <axis xyz="-0.0 -0.707107 -0.707107"/>
-  <limit upper="0.349066" lower="-0.349066" effort="1000" velocity="100"/>
-</joint>
-<joint name="fins_rev4" type="revolute">
-<!-- <joint name="fins_rev4" type="fixed"> -->
-  <origin xyz="-1.700844 -0.127279 0.127279" rpy="0 0 0"/>
-  <parent link="base_link"/>
-  <child link="FinHolder_4"/>
-  <axis xyz="-0.0 -0.707107 0.707107"/>
-  <limit upper="0.349066" lower="-0.349066" effort="1000" velocity="100"/>
-</joint>
-<!-- <joint name="wings_fold1" type="revolute"> -->
-<joint name="wings_fold1" type="fixed">
-  <origin xyz="-0.380856 0.163355 0.163355" rpy="0 0 0"/>
-  <parent link="base_link"/>
-  <child link="Wing1_1"/>
-  <!-- <axis xyz="1.0 -0.0 -0.0"/> -->
-  <!-- <limit upper="2.146755" lower="0.0" effort="100" velocity="100"/> -->
-</joint>
-<!-- <joint name="wings_fold2" type="revolute"> -->
-<joint name="wings_fold2" type="fixed">
-  <origin xyz="-0.380856 0.163355 -0.163355" rpy="0 0 0"/>
-  <parent link="base_link"/>
-  <child link="Wing1_2"/>
-  <!-- <axis xyz="1.0 0.0 -0.0"/> -->
-  <!-- <limit upper="2.146755" lower="0.0" effort="100" velocity="100"/> -->
-</joint>
-<!-- <joint name="wings_fold3" type="revolute"> -->
-<joint name="wings_fold3" type="fixed">
-  <origin xyz="-0.380856 -0.163355 -0.163355" rpy="0 0 0"/>
-  <parent link="base_link"/>
-  <child link="Wing1_3"/>
-  <!-- <axis xyz="1.0 0.0 -0.0"/> -->
-  <!-- <limit upper="2.146755" lower="0.0" effort="100" velocity="100"/> -->
-</joint>
-<!-- <joint name="wings_fold4" type="revolute"> -->
-<joint name="wings_fold4" type="fixed">
-  <origin xyz="-0.380856 -0.163355 0.163355" rpy="0 0 0"/>
-  <parent link="base_link"/>
-  <child link="Wing1_4"/>
-  <!-- <axis xyz="1.0 -0.0 -0.0"/> -->
-  <!-- <limit upper="2.146755" lower="0.0" effort="100" velocity="100"/> -->
-</joint>
-<!-- <joint name="fin_fold1" type="revolute"> -->
-<joint name="fin_fold1" type="fixed">
-  <origin xyz="0.0 0.038891 0.038891" rpy="0 0 0"/>
-  <parent link="FinHolder_1"/>
-  <child link="Fin_1"/>
-  <!-- <axis xyz="1.0 0.0 0.0"/> -->
-  <!-- <limit upper="2.146755" lower="0.0" effort="100" velocity="100"/> -->
-</joint>
-<!-- <joint name="fin_fold2" type="revolute"> -->
-<joint name="fin_fold2" type="fixed">
-  <origin xyz="0.0 0.038879 -0.038903" rpy="0 0 0"/>
-  <parent link="FinHolder_2"/>
-  <child link="Fin_2"/>
-  <!-- <axis xyz="1.0 0.0 -0.0"/> -->
-  <!-- <limit upper="2.146755" lower="0.0" effort="100" velocity="100"/> -->
-</joint>
-<!-- <joint name="fin_fold3" type="revolute"> -->
-<joint name="fin_fold3" type="fixed">
-  <origin xyz="0.0 -0.038891 -0.038891" rpy="0 0 0"/>
-  <parent link="FinHolder_3"/>
-  <child link="Fin_3"/>
-  <!-- <axis xyz="1.0 -0.0 -0.0"/> -->
-  <!-- <limit upper="2.146755" lower="0.0" effort="100" velocity="100"/> -->
-</joint>
-<!-- <joint name="fin_fold4" type="revolute"> -->
-<joint name="fin_fold4" type="fixed">
-  <origin xyz="0.0 -0.038891 0.038891" rpy="0 0 0"/>
-  <parent link="FinHolder_4"/>
-  <child link="Fin_4"/>
-  <!-- <axis xyz="1.0 -0.0 0.0"/> -->
-  <!-- <limit upper="2.146755" lower="0.0" effort="100" velocity="100"/> -->
-</joint>
+<xacro:if value="${deflection}">
+  <joint name="fins_rev1" type="revolute">
+    <origin xyz="-1.700844 0.127279 0.127279" rpy="0 0 0"/>
+    <parent link="base_link"/>
+    <child link="FinHolder_1"/>
+    <axis xyz="-0.0 0.707107 0.707107"/>
+    <limit upper="0.349066" lower="-0.349066" effort="1000" velocity="100"/>
+  </joint>
+  <joint name="fins_rev2" type="revolute">
+    <origin xyz="-1.700844 0.127279 -0.127279" rpy="0 0 0"/>
+    <parent link="base_link"/>
+    <child link="FinHolder_2"/>
+    <axis xyz="-0.0 0.707107 -0.707107"/>
+    <limit upper="0.349066" lower="-0.349066" effort="1000" velocity="100"/>
+  </joint>
+  <joint name="fins_rev3" type="revolute">
+    <origin xyz="-1.700844 -0.127279 -0.127279" rpy="0 0 0"/>
+    <parent link="base_link"/>
+    <child link="FinHolder_3"/>
+    <axis xyz="-0.0 -0.707107 -0.707107"/>
+    <limit upper="0.349066" lower="-0.349066" effort="1000" velocity="100"/>
+  </joint>
+  <joint name="fins_rev4" type="revolute">
+    <origin xyz="-1.700844 -0.127279 0.127279" rpy="0 0 0"/>
+    <parent link="base_link"/>
+    <child link="FinHolder_4"/>
+    <axis xyz="-0.0 -0.707107 0.707107"/>
+    <limit upper="0.349066" lower="-0.349066" effort="1000" velocity="100"/>
+  </joint>
+</xacro:if>
+<xacro:unless value="${deflection}">
+  <joint name="fins_rev1" type="fixed">
+    <origin xyz="-1.700844 0.127279 0.127279" rpy="0 0 0"/>
+    <parent link="base_link"/>
+    <child link="FinHolder_1"/>
+  </joint>
+  <joint name="fins_rev2" type="fixed">
+    <origin xyz="-1.700844 0.127279 -0.127279" rpy="0 0 0"/>
+    <parent link="base_link"/>
+    <child link="FinHolder_2"/>
+  </joint>
+  <joint name="fins_rev3" type="fixed">
+    <origin xyz="-1.700844 -0.127279 -0.127279" rpy="0 0 0"/>
+    <parent link="base_link"/>
+    <child link="FinHolder_3"/>
+  </joint>
+  <joint name="fins_rev4" type="fixed">
+    <origin xyz="-1.700844 -0.127279 0.127279" rpy="0 0 0"/>
+    <parent link="base_link"/>
+    <child link="FinHolder_4"/>
+  </joint>
+</xacro:unless>
+<xacro:if value="${foldable}">
+  <joint name="wings_fold1" type="revolute">
+    <origin xyz="-0.380856 0.163355 0.163355" rpy="0 0 0"/>
+    <parent link="base_link"/>
+    <child link="Wing1_1"/>
+    <axis xyz="1.0 -0.0 -0.0"/>
+    <limit upper="2.146755" lower="0.0" effort="100" velocity="100"/>
+  </joint>
+  <joint name="wings_fold2" type="revolute">
+    <origin xyz="-0.380856 0.163355 -0.163355" rpy="0 0 0"/>
+    <parent link="base_link"/>
+    <child link="Wing1_2"/>
+    <axis xyz="1.0 0.0 -0.0"/>
+    <limit upper="2.146755" lower="0.0" effort="100" velocity="100"/>
+  </joint>
+  <joint name="wings_fold3" type="revolute">
+    <origin xyz="-0.380856 -0.163355 -0.163355" rpy="0 0 0"/>
+    <parent link="base_link"/>
+    <child link="Wing1_3"/>
+    <axis xyz="1.0 0.0 -0.0"/>
+    <limit upper="2.146755" lower="0.0" effort="100" velocity="100"/>
+  </joint>
+  <joint name="wings_fold4" type="revolute">
+    <origin xyz="-0.380856 -0.163355 0.163355" rpy="0 0 0"/>
+    <parent link="base_link"/>
+    <child link="Wing1_4"/>
+    <axis xyz="1.0 -0.0 -0.0"/>
+    <limit upper="2.146755" lower="0.0" effort="100" velocity="100"/>
+  </joint>
+  <joint name="fin_fold1" type="revolute">
+    <origin xyz="0.0 0.038891 0.038891" rpy="0 0 0"/>
+    <parent link="FinHolder_1"/>
+    <child link="Fin_1"/>
+    <axis xyz="1.0 0.0 0.0"/>
+    <limit upper="2.146755" lower="0.0" effort="100" velocity="100"/>
+  </joint>
+  <joint name="fin_fold2" type="revolute">
+    <origin xyz="0.0 0.038879 -0.038903" rpy="0 0 0"/>
+    <parent link="FinHolder_2"/>
+    <child link="Fin_2"/>
+    <axis xyz="1.0 0.0 -0.0"/>
+    <limit upper="2.146755" lower="0.0" effort="100" velocity="100"/>
+  </joint>
+  <joint name="fin_fold3" type="revolute">
+    <origin xyz="0.0 -0.038891 -0.038891" rpy="0 0 0"/>
+    <parent link="FinHolder_3"/>
+    <child link="Fin_3"/>
+    <axis xyz="1.0 -0.0 -0.0"/>
+    <limit upper="2.146755" lower="0.0" effort="100" velocity="100"/>
+  </joint>
+  <joint name="fin_fold4" type="revolute">
+    <origin xyz="0.0 -0.038891 0.038891" rpy="0 0 0"/>
+    <parent link="FinHolder_4"/>
+    <child link="Fin_4"/>
+    <axis xyz="1.0 -0.0 0.0"/>
+    <limit upper="2.146755" lower="0.0" effort="100" velocity="100"/>
+  </joint>
+</xacro:if>
+<xacro:unless value="${foldable}">
+    <joint name="wings_fold1" type="fixed">
+      <origin xyz="-0.380856 0.163355 0.163355" rpy="0 0 0"/>
+      <parent link="base_link"/>
+      <child link="Wing1_1"/>
+    </joint>
+    <joint name="wings_fold2" type="fixed">
+      <origin xyz="-0.380856 0.163355 -0.163355" rpy="0 0 0"/>
+      <parent link="base_link"/>
+      <child link="Wing1_2"/>
+    </joint>
+    <joint name="wings_fold3" type="fixed">
+      <origin xyz="-0.380856 -0.163355 -0.163355" rpy="0 0 0"/>
+      <parent link="base_link"/>
+      <child link="Wing1_3"/>
+    </joint>
+    <joint name="wings_fold4" type="fixed">
+      <origin xyz="-0.380856 -0.163355 0.163355" rpy="0 0 0"/>
+      <parent link="base_link"/>
+      <child link="Wing1_4"/>
+    </joint>
+    <joint name="fin_fold1" type="fixed">
+      <origin xyz="0.0 0.038891 0.038891" rpy="0 0 0"/>
+      <parent link="FinHolder_1"/>
+      <child link="Fin_1"/>
+    </joint>
+    <joint name="fin_fold2" type="fixed">
+      <origin xyz="0.0 0.038879 -0.038903" rpy="0 0 0"/>
+      <parent link="FinHolder_2"/>
+      <child link="Fin_2"/>
+    </joint>
+    <joint name="fin_fold3" type="fixed">
+      <origin xyz="0.0 -0.038891 -0.038891" rpy="0 0 0"/>
+      <parent link="FinHolder_3"/>
+      <child link="Fin_3"/>
+    </joint>
+    <joint name="fin_fold4" type="fixed">
+      <origin xyz="0.0 -0.038891 0.038891" rpy="0 0 0"/>
+      <parent link="FinHolder_4"/>
+      <child link="Fin_4"/>
+    </joint>
+</xacro:unless>
 <xacro:if value="${use_holder}">
   <joint name="HolderJoint1" type="fixed">

Commit message: deflexion test

File: src/ssm_models/model_missile_description/model_missile.urdf (robot description, URDF)
Before this commit: robot model_missile, 13 links, 12 joints
Joints:
- joint fin_fold1: axis 1.0 0.0 0.0 -> (none); limit lower=0.0 upper=2.146755 effort=100 velocity=100 -> (none); type revolute -> fixed
- joint fin_fold2: axis 1.0 0.0 -0.0 -> (none); limit lower=0.0 upper=2.146755 effort=100 velocity=100 -> (none); type revolute -> fixed
- joint fin_fold3: axis 1.0 -0.0 -0.0 -> (none); limit lower=0.0 upper=2.146755 effort=100 velocity=100 -> (none); type revolute -> fixed
- joint fin_fold4: axis 1.0 -0.0 0.0 -> (none); limit lower=0.0 upper=2.146755 effort=100 velocity=100 -> (none); type revolute -> fixed
- joint fins_rev1: limit lower=-0.349066 upper=0.349066 effort=1000 velocity=100 -> lower=-0.349066 upper=0.349066 effort=1000000 velocity=1000000
- joint fins_rev2: limit lower=-0.349066 upper=0.349066 effort=1000 velocity=100 -> lower=-0.349066 upper=0.349066 effort=1000000 velocity=1000000
- joint fins_rev3: limit lower=-0.349066 upper=0.349066 effort=1000 velocity=100 -> lower=-0.349066 upper=0.349066 effort=1000000 velocity=1000000
- joint fins_rev4: limit lower=-0.349066 upper=0.349066 effort=1000 velocity=100 -> lower=-0.349066 upper=0.349066 effort=1000000 velocity=1000000
- joint wings_fold1: axis 1.0 -0.0 -0.0 -> (none); limit lower=0.0 upper=2.146755 effort=100 velocity=100 -> (none); type revolute -> fixed
- joint wings_fold2: axis 1.0 0.0 -0.0 -> (none); limit lower=0.0 upper=2.146755 effort=100 velocity=100 -> (none); type revolute -> fixed
- joint wings_fold3: axis 1.0 0.0 -0.0 -> (none); limit lower=0.0 upper=2.146755 effort=100 velocity=100 -> (none); type revolute -> fixed
- joint wings_fold4: axis 1.0 -0.0 -0.0 -> (none); limit lower=0.0 upper=2.146755 effort=100 velocity=100 -> (none); type revolute -> fixed

File: src/ssm_models/model_missile_description/urdf/model_missile.xacro (robot description, xacro)
@@ -3,5 +3,5 @@
 <xacro:property name="use_booster" value="false"/>
 <xacro:property name="use_holder" value="false"/>
-<xacro:property name="foldable" value="true"/>
+<xacro:property name="foldable" value="false"/>
 <xacro:property name="deflection" value="true"/>
 <xacro:include filename="$(find model_missile_description)/urdf/materials.xacro" />
@@ -385,5 +385,6 @@
     <child link="FinHolder_1"/>
     <axis xyz="-0.0 0.707107 0.707107"/>
-    <limit upper="0.349066" lower="-0.349066" effort="1000" velocity="100"/>
+    <limit upper="0.349066" lower="-0.349066" effort="10000000" velocity="1000000"/>
+    <dynamics damping="5"/>
   </joint>
   <joint name="fins_rev2" type="revolute">
@@ -392,5 +393,6 @@
     <child link="FinHolder_2"/>
     <axis xyz="-0.0 0.707107 -0.707107"/>
-    <limit upper="0.349066" lower="-0.349066" effort="1000" velocity="100"/>
+    <limit upper="0.349066" lower="-0.349066" effort="10000000" velocity="1000000"/>
+    <dynamics damping="5"/>
   </joint>
   <joint name="fins_rev3" type="revolute">
@@ -399,5 +401,6 @@
     <child link="FinHolder_3"/>
     <axis xyz="-0.0 -0.707107 -0.707107"/>
-    <limit upper="0.349066" lower="-0.349066" effort="1000" velocity="100"/>
+    <limit upper="0.349066" lower="-0.349066" effort="10000000" velocity="1000000"/>
+    <dynamics damping="5"/>
   </joint>
   <joint name="fins_rev4" type="revolute">
@@ -406,5 +409,6 @@
     <child link="FinHolder_4"/>
     <axis xyz="-0.0 -0.707107 0.707107"/>
-    <limit upper="0.349066" lower="-0.349066" effort="1000" velocity="100"/>
+    <limit upper="0.349066" lower="-0.349066" effort="10000000" velocity="1000000"/>
+    <dynamics damping="5"/>
   </joint>
 </xacro:if>
