Commit message: detachable and foldable test successfull

File: src/ssm_models/model_missile_description/urdf/model_missile.xacro (robot description, xacro)
@@ -1,6 +1,6 @@
 <?xml version="1.0" ?>
 <robot name="model_missile" xmlns:xacro="http://www.ros.org/wiki/xacro">
-<xacro:property name="use_booster" value="false"/>
-<xacro:property name="use_holder" value="false"/>
+<xacro:property name="use_booster" value="true"/>
+<xacro:property name="use_holder" value="true"/>
 <xacro:include filename="$(find model_missile_description)/urdf/materials.xacro" />
 <xacro:include filename="$(find model_missile_description)/urdf/model_missile.trans" />

Commit message: test aerodynamic on fins fixed

File: src/ssm_models/model_missile_description/urdf/model_missile.xacro (robot description, xacro)
@@ -377,87 +377,99 @@
   </joint>
 </xacro:if>
-<joint name="fins_rev1" type="revolute">
+<!-- <joint name="fins_rev1" type="revolute"> -->
+<joint name="fins_rev1" type="fixed">
   <origin xyz="-1.700844 0.127279 0.127279" rpy="0 0 0"/>
   <parent link="base_link"/>
   <child link="FinHolder_1"/>
-  <axis xyz="-0.0 0.707107 0.707107"/>
-  <limit upper="0.349066" lower="-0.349066" effort="100" velocity="100"/>
-</joint>
-<joint name="fins_rev4" type="revolute">
+  <!-- <axis xyz="-0.0 0.707107 0.707107"/> -->
+  <!-- <limit upper="0.349066" lower="-0.349066" effort="100" velocity="100"/> -->
+</joint>
+<!-- <joint name="fins_rev2" type="revolute"> -->
+<joint name="fins_rev2" type="fixed">
+  <origin xyz="-1.700844 0.127279 -0.127279" rpy="0 0 0"/>
+  <parent link="base_link"/>
+  <child link="FinHolder_2"/>
+  <!-- <axis xyz="-0.0 0.707107 -0.707107"/> -->
+  <!-- <limit upper="0.349066" lower="-0.349066" effort="100" velocity="100"/> -->
+</joint>
+<!-- <joint name="fins_rev3" type="revolute"> -->
+<joint name="fins_rev3" type="fixed">
+  <origin xyz="-1.700844 -0.127279 -0.127279" rpy="0 0 0"/>
+  <parent link="base_link"/>
+  <child link="FinHolder_3"/>
+  <!-- <axis xyz="-0.0 -0.707107 -0.707107"/> -->
+  <!-- <limit upper="0.349066" lower="-0.349066" effort="100" velocity="100"/> -->
+</joint>
+<!-- <joint name="fins_rev4" type="revolute"> -->
+<joint name="fins_rev4" type="fixed">
   <origin xyz="-1.700844 -0.127279 0.127279" rpy="0 0 0"/>
   <parent link="base_link"/>
   <child link="FinHolder_4"/>
-  <axis xyz="-0.0 -0.707107 0.707107"/>
-  <limit upper="0.349066" lower="-0.349066" effort="100" velocity="100"/>
-</joint>
-<joint name="fins_rev3" type="revolute">
-  <origin xyz="-1.700844 -0.127279 -0.127279" rpy="0 0 0"/>
-  <parent link="base_link"/>
-  <child link="FinHolder_3"/>
-  <axis xyz="-0.0 -0.707107 -0.707107"/>
-  <limit upper="0.349066" lower="-0.349066" effort="100" velocity="100"/>
-</joint>
-<joint name="fins_rev2" type="revolute">
-  <origin xyz="-1.700844 0.127279 -0.127279" rpy="0 0 0"/>
-  <parent link="base_link"/>
-  <child link="FinHolder_2"/>
-  <axis xyz="-0.0 0.707107 -0.707107"/>
-  <limit upper="0.349066" lower="-0.349066" effort="100" velocity="100"/>
-</joint>
-<joint name="wings_fold1" type="revolute">
+  <!-- <axis xyz="-0.0 -0.707107 0.707107"/> -->
+  <!-- <limit upper="0.349066" lower="-0.349066" effort="100" velocity="100"/> -->
+</joint>
+<!-- <joint name="wings_fold1" type="revolute"> -->
+<joint name="wings_fold1" type="fixed">
   <origin xyz="-0.380856 0.163355 0.163355" rpy="0 0 0"/>
   <parent link="base_link"/>
   <child link="Wing1_1"/>
-  <axis xyz="1.0 -0.0 -0.0"/>
-  <limit upper="2.146755" lower="0.0" effort="100" velocity="100"/>
-</joint>
-<joint name="wings_fold2" type="revolute">
+  <!-- <axis xyz="1.0 -0.0 -0.0"/> -->
+  <!-- <limit upper="2.146755" lower="0.0" effort="100" velocity="100"/> -->
+</joint>
+<!-- <joint name="wings_fold2" type="revolute"> -->
+<joint name="wings_fold2" type="fixed">
   <origin xyz="-0.380856 0.163355 -0.163355" rpy="0 0 0"/>
   <parent link="base_link"/>
   <child link="Wing1_2"/>
-  <axis xyz="1.0 0.0 -0.0"/>
-  <limit upper="2.146755" lower="0.0" effort="100" velocity="100"/>
-</joint>
-<joint name="wings_fold3" type="revolute">
+  <!-- <axis xyz="1.0 0.0 -0.0"/> -->
+  <!-- <limit upper="2.146755" lower="0.0" effort="100" velocity="100"/> -->
+</joint>
+<!-- <joint name="wings_fold3" type="revolute"> -->
+<joint name="wings_fold3" type="fixed">
   <origin xyz="-0.380856 -0.163355 -0.163355" rpy="0 0 0"/>
   <parent link="base_link"/>
   <child link="Wing1_3"/>
-  <axis xyz="1.0 0.0 -0.0"/>
-  <limit upper="2.146755" lower="0.0" effort="100" velocity="100"/>
-</joint>
-<joint name="wings_fold4" type="revolute">
+  <!-- <axis xyz="1.0 0.0 -0.0"/> -->
+  <!-- <limit upper="2.146755" lower="0.0" effort="100" velocity="100"/> -->
+</joint>
+<!-- <joint name="wings_fold4" type="revolute"> -->
+<joint name="wings_fold4" type="fixed">
   <origin xyz="-0.380856 -0.163355 0.163355" rpy="0 0 0"/>
   <parent link="base_link"/>
   <child link="Wing1_4"/>
-  <axis xyz="1.0 -0.0 -0.0"/>
-  <limit upper="2.146755" lower="0.0" effort="100" velocity="100"/>
-</joint>
-<joint name="fin_fold1" type="revolute">
+  <!-- <axis xyz="1.0 -0.0 -0.0"/> -->
+  <!-- <limit upper="2.146755" lower="0.0" effort="100" velocity="100"/> -->
+</joint>
+<!-- <joint name="fin_fold1" type="revolute"> -->
+<joint name="fin_fold1" type="fixed">
   <origin xyz="0.0 0.038891 0.038891" rpy="0 0 0"/>
   <parent link="FinHolder_1"/>
   <child link="Fin_1"/>
-  <axis xyz="1.0 0.0 0.0"/>
-  <limit upper="2.146755" lower="0.0" effort="100" velocity="100"/>
-</joint>
-<joint name="fin_fold2" type="revolute">
+  <!-- <axis xyz="1.0 0.0 0.0"/> -->
+  <!-- <limit upper="2.146755" lower="0.0" effort="100" velocity="100"/> -->
+</joint>
+<!-- <joint name="fin_fold2" type="revolute"> -->
+<joint name="fin_fold2" type="fixed">
   <origin xyz="0.0 0.038879 -0.038903" rpy="0 0 0"/>
   <parent link="FinHolder_2"/>
   <child link="Fin_2"/>
-  <axis xyz="1.0 0.0 -0.0"/>
-  <limit upper="2.146755" lower="0.0" effort="100" velocity="100"/>
-</joint>
-<joint name="fin_fold3" type="revolute">
+  <!-- <axis xyz="1.0 0.0 -0.0"/> -->
+  <!-- <limit upper="2.146755" lower="0.0" effort="100" velocity="100"/> -->
+</joint>
+<!-- <joint name="fin_fold3" type="revolute"> -->
+<joint name="fin_fold3" type="fixed">
   <origin xyz="0.0 -0.038891 -0.038891" rpy="0 0 0"/>
   <parent link="FinHolder_3"/>
   <child link="Fin_3"/>
-  <axis xyz="1.0 -0.0 -0.0"/>
-  <limit upper="2.146755" lower="0.0" effort="100" velocity="100"/>
-</joint>
-<joint name="fin_fold4" type="revolute">
+  <!-- <axis xyz="1.0 -0.0 -0.0"/> -->
+  <!-- <limit upper="2.146755" lower="0.0" effort="100" velocity="100"/> -->
+</joint>
+<!-- <joint name="fin_fold4" type="revolute"> -->
+<joint name="fin_fold4" type="fixed">
   <origin xyz="0.0 -0.038891 0.038891" rpy="0 0 0"/>
   <parent link="FinHolder_4"/>
   <child link="Fin_4"/>
-  <axis xyz="1.0 -0.0 0.0"/>
-  <limit upper="2.146755" lower="0.0" effort="100" velocity="100"/>
+  <!-- <axis xyz="1.0 -0.0 0.0"/> -->
+  <!-- <limit upper="2.146755" lower="0.0" effort="100" velocity="100"/> -->
 </joint>
 <xacro:if value="${use_holder}">

Commit message: deflexion test unfinished

File: src/ssm_models/model_missile_description/urdf/model_missile.xacro (robot description, xacro)
@@ -377,35 +377,35 @@
   </joint>
 </xacro:if>
-<!-- <joint name="fins_rev1" type="revolute"> -->
-<joint name="fins_rev1" type="fixed">
+<joint name="fins_rev1" type="revolute">
+<!-- <joint name="fins_rev1" type="fixed"> -->
   <origin xyz="-1.700844 0.127279 0.127279" rpy="0 0 0"/>
   <parent link="base_link"/>
   <child link="FinHolder_1"/>
-  <!-- <axis xyz="-0.0 0.707107 0.707107"/> -->
-  <!-- <limit upper="0.349066" lower="-0.349066" effort="100" velocity="100"/> -->
-</joint>
-<!-- <joint name="fins_rev2" type="revolute"> -->
-<joint name="fins_rev2" type="fixed">
+  <axis xyz="-0.0 0.707107 0.707107"/>
+  <limit upper="0.349066" lower="-0.349066" effort="1000" velocity="100"/>
+</joint>
+<joint name="fins_rev2" type="revolute">
+<!-- <joint name="fins_rev2" type="fixed"> -->
   <origin xyz="-1.700844 0.127279 -0.127279" rpy="0 0 0"/>
   <parent link="base_link"/>
   <child link="FinHolder_2"/>
-  <!-- <axis xyz="-0.0 0.707107 -0.707107"/> -->
-  <!-- <limit upper="0.349066" lower="-0.349066" effort="100" velocity="100"/> -->
-</joint>
-<!-- <joint name="fins_rev3" type="revolute"> -->
-<joint name="fins_rev3" type="fixed">
+  <axis xyz="-0.0 0.707107 -0.707107"/>
+  <limit upper="0.349066" lower="-0.349066" effort="1000" velocity="100"/>
+</joint>
+<joint name="fins_rev3" type="revolute">
+<!-- <joint name="fins_rev3" type="fixed"> -->
   <origin xyz="-1.700844 -0.127279 -0.127279" rpy="0 0 0"/>
   <parent link="base_link"/>
   <child link="FinHolder_3"/>
-  <!-- <axis xyz="-0.0 -0.707107 -0.707107"/> -->
-  <!-- <limit upper="0.349066" lower="-0.349066" effort="100" velocity="100"/> -->
-</joint>
-<!-- <joint name="fins_rev4" type="revolute"> -->
-<joint name="fins_rev4" type="fixed">
+  <axis xyz="-0.0 -0.707107 -0.707107"/>
+  <limit upper="0.349066" lower="-0.349066" effort="1000" velocity="100"/>
+</joint>
+<joint name="fins_rev4" type="revolute">
+<!-- <joint name="fins_rev4" type="fixed"> -->
   <origin xyz="-1.700844 -0.127279 0.127279" rpy="0 0 0"/>
   <parent link="base_link"/>
   <child link="FinHolder_4"/>
-  <!-- <axis xyz="-0.0 -0.707107 0.707107"/> -->
-  <!-- <limit upper="0.349066" lower="-0.349066" effort="100" velocity="100"/> -->
+  <axis xyz="-0.0 -0.707107 0.707107"/>
+  <limit upper="0.349066" lower="-0.349066" effort="1000" velocity="100"/>
 </joint>
 <!-- <joint name="wings_fold1" type="revolute"> -->

Commit message: deflexion

File: src/ssm_models/model_missile_description/urdf/model_missile.xacro (robot description, xacro)
@@ -385,6 +385,6 @@
     <child link="FinHolder_1"/>
     <axis xyz="-0.0 0.707107 0.707107"/>
-    <limit upper="0.349066" lower="-0.349066" effort="10000000" velocity="1000000"/>
-    <dynamics damping="5"/>
+    <limit upper="0.349066" lower="-0.349066" effort="90000000" velocity="90000000"/>
+    <dynamics damping="7"/>
   </joint>
   <joint name="fins_rev2" type="revolute">
@@ -393,6 +393,6 @@
     <child link="FinHolder_2"/>
     <axis xyz="-0.0 0.707107 -0.707107"/>
-    <limit upper="0.349066" lower="-0.349066" effort="10000000" velocity="1000000"/>
-    <dynamics damping="5"/>
+    <limit upper="0.349066" lower="-0.349066" effort="90000000" velocity="90000000"/>
+    <dynamics damping="7"/>
   </joint>
   <joint name="fins_rev3" type="revolute">
@@ -401,6 +401,6 @@
     <child link="FinHolder_3"/>
     <axis xyz="-0.0 -0.707107 -0.707107"/>
-    <limit upper="0.349066" lower="-0.349066" effort="10000000" velocity="1000000"/>
-    <dynamics damping="5"/>
+    <limit upper="0.349066" lower="-0.349066" effort="90000000" velocity="90000000"/>
+    <dynamics damping="7"/>
   </joint>
   <joint name="fins_rev4" type="revolute">
@@ -409,6 +409,6 @@
     <child link="FinHolder_4"/>
     <axis xyz="-0.0 -0.707107 0.707107"/>
-    <limit upper="0.349066" lower="-0.349066" effort="10000000" velocity="1000000"/>
-    <dynamics damping="5"/>
+    <limit upper="0.349066" lower="-0.349066" effort="90000000" velocity="90000000"/>
+    <dynamics damping="7"/>
   </joint>
 </xacro:if>
