Commit message: To Preset

File: src/ssm_models/launcher20deg_description/launcher20deg.urdf (robot description, URDF)
Before this commit: robot launcher20deg, 7 links, 6 joints
Links:
- removed link Cup_3
Joints:
- removed joint CupOpener

File: src/ssm_models/missile_description/urdf/materials.xacro (robot description, xacro)
@@ -1,6 +1,30 @@
 <?xml version="1.0" ?>
-<robot name="missile" xmlns:xacro="http://www.ros.org/wiki/xacro" >
-<material name="silver">
-  <color rgba="0.700 0.700 0.700 1.000"/>
-</material>
+<robot name="model_missile" xmlns:xacro="http://www.ros.org/wiki/xacro" >
+  <material name="grey">
+    <color rgba="${211/256} ${211/256} ${211/256} 1.0"/>
+  </material>
+  <material name="darkgrey">
+    <color rgba="${47/255} ${79/255} ${79/255} 1.000"/>
+  </material>
+  <material name="silver">
+    <color rgba="0.700 0.700 0.700 1.000"/>
+  </material>
+  <material name="white">
+    <color rgba="1 1 1 1" />
+  </material>
+  <material name="orange">
+    <color rgba="1 0.3 0.1 1"/>
+  </material>
+  <material name="blue">
+    <color rgba="0.2 0.2 1 1"/>
+  </material>
+  <material name="red">
+    <color rgba="0.8 0 0 1"/>
+  </material>
+  <material name="green">
+    <color rgba="0.0 1 0.0 1"/>
+  </material>
+  <material name="black">
+    <color rgba="0 0 0 1"/>
+  </material>
 </robot>

File: src/ssm_models/missile_description/urdf/missile.xacro (robot description, xacro)
@@ -1,4 +1,8 @@
 <?xml version="1.0" ?>
 <robot name="missile" xmlns:xacro="http://www.ros.org/wiki/xacro">
+<xacro:property name="use_booster" value="true"/>
+<xacro:property name="use_holder" value="true"/>
+<xacro:property name="foldable" value="true"/>
+<xacro:property name="deflection" value="true"/>
 <xacro:include filename="$(find missile_description)/urdf/materials.xacro" />
 <xacro:include filename="$(find missile_description)/urdf/missile.trans" />
